Commit message: base_link used in xacro

File: gz_models/models/urdf/diff_drive.xacro (robot description, xacro)
@@ -53,4 +53,5 @@
         </joint>
     </xacro:macro>
+    <link name="base_link"></link>
     <!-- Chassis -->
     <link name="chassis">
@@ -75,4 +76,9 @@
         </collision>
     </link>
+    <joint name="chassis_joint" type="fixed">
+        <parent link="base_link"/>
+        <child link="chassis"/>
+        <origin xyz="0 0 0" rpy="0 0 0" />
+    </joint>
     <!-- Instantiate wheels -->
     <xacro:wheel name="left" side="1" />

Commit message: odometry wrong display in rviz fixed

File: gz_models/models/urdf/diff_drive.xacro (robot description, xacro)
@@ -77,6 +77,6 @@
     </link>
     <joint name="chassis_joint" type="fixed">
-        <parent link="base_link"/>
-        <child link="chassis"/>
+        <parent link="base_link" />
+        <child link="chassis" />
         <origin xyz="0 0 0" rpy="0 0 0" />
     </joint>
@@ -158,5 +158,5 @@
             name="gz::sim::systems::JointStatePublisher">
         </plugin>
-        <plugin
+        <!-- <plugin
             filename="gz-sim-pose-publisher-system"
             name="gz::sim::systems::PosePublisher">
@@ -165,10 +165,11 @@
             <static_publisher>true</static_publisher>
             <static_update_frequency>1</static_update_frequency>
-        </plugin>
+        </plugin> -->
         <plugin
             filename="gz-sim-odometry-publisher-system"
             name="gz::sim::systems::OdometryPublisher">
-            <odom_frame>$(arg robot_model_name)/odom</odom_frame>
-            <robot_base_frame>$(arg robot_model_name)</robot_base_frame>
+            <odom_frame>$(arg robot_model_name)_odom</odom_frame>
+            <robot_base_frame>$(arg robot_model_name)/base_link</robot_base_frame>
+            <odom_publish_frequency>20</odom_publish_frequency>
         </plugin>
     </gazebo>

Commit message: wall static=true; diff_drive odom error fixed

File: gz_models/models/urdf/diff_drive.xacro (robot description, xacro)
@@ -37,5 +37,5 @@
                 </material>
             </visual>
-            <collision>
+            <collision name="wheel_collision">
                 <origin xyz="0 0 0" rpy="0 0 0" />
                 <geometry>
@@ -52,4 +52,14 @@
             <limit lower="-1.79769e+308" upper="1.79769e+308" effort="1000.0" velocity="50.0" />
         </joint>
+        <!-- <gazebo reference="${name}_wheel">
+            <sensor name="contact_sensor" type="contact">
+                <always_on>true</always_on>
+                <update_rate>30.0</update_rate>
+                <topic>${name}_wheel_contacts</topic>
+                <contact>
+                    <collision>wheel_collision</collision>
+                </contact>
+            </sensor>
+        </gazebo> -->
     </xacro:macro>
     <link name="base_link"></link>
@@ -145,4 +155,5 @@
             <wheel_radius>${wheel_radius}</wheel_radius>
             <odom_publish_frequency>1</odom_publish_frequency>
+            <odom_topic>model/$(arg robot_model_name)/diffdrive_plugin/odom</odom_topic>
             <max_linear_acceleration>1</max_linear_acceleration>
             <min_linear_acceleration>-1</min_linear_acceleration>
@@ -169,5 +180,5 @@
             filename="gz-sim-odometry-publisher-system"
             name="gz::sim::systems::OdometryPublisher">
-            <odom_frame>$(arg robot_model_name)_odom</odom_frame>
+            <odom_frame>$(arg robot_model_name)/odom</odom_frame>
             <robot_base_frame>$(arg robot_model_name)/base_link</robot_base_frame>
             <odom_publish_frequency>20</odom_publish_frequency>
@@ -176,5 +187,5 @@
     <!-- Gazebo Sensor for Lidar -->
     <gazebo reference="lidar_link">
-        <sensor name="gpu_lidar" type="gpu_lidar">
+        <sensor name="my_lidar" type="gpu_lidar">
             <pose>0 0 0 0 0 0</pose>
             <topic>/model/$(arg robot_model_name)/scan</topic>

File: gz_models/models/urdf/wall.xacro (robot description, xacro)
@@ -6,16 +6,27 @@
     <xacro:property name="visual_size" value="0.5 10.0 2.0" />
     <xacro:property name="color" value="1.0 1.0 0.0 1" />
+    <xacro:property name="color_name" value="yellow" />
     <xacro:property name="mass" value="1.14395" />
     <xacro:property name="ixx" value="9.532917" />
     <xacro:property name="iyy" value="0.023832" />
     <xacro:property name="izz" value="9.556749" />
-    <xacro:macro name="touch_plugin" params="target">
-        <plugin name="touch_${target}" filename="gz-sim-touchplugin-system">
+    <!-- <xacro:macro name="touch_plugin" params="target">
+        <plugin filename="gz-sim-touchplugin-system"
+            name="gz::sim::systems::TouchPlugin">
             <target>${target}</target>
             <namespace>wall</namespace>
-            <time>0.1</time>
+            <time>0.0001</time>
             <enabled>true</enabled>
         </plugin>
-    </xacro:macro>
+        <plugin filename="gz-sim-triggered-publisher-system"
+            name="gz::sim::systems::TriggeredPublisher">
+            <input type="gz.msgs.Boolean" topic="/wall/touched">
+                <match>data: true</match>
+            </input>
+            <output type="gz.msgs.Twist" topic="/model/${target}/cmd_vel">
+                linear: {x: 0.0}, angular: {z: 0.0}
+            </output>
+        </plugin>
+    </xacro:macro> -->
     <link name="${link_name}">
         <inertial>
@@ -28,9 +39,9 @@
                 <box size="${visual_size}" />
             </geometry>
-            <material name="blue">
+            <material name="${color_name}">
                 <color rgba="${color}" />
             </material>
         </visual>
-        <collision>
+        <collision name="wall_collision">
             <origin xyz="0 0 0" rpy="0 0 0" />
             <geometry>
@@ -39,19 +50,15 @@
         </collision>
     </link>
-    <gazebo reference="${link_name}">
-        <!-- Contact sensor -->
-        <sensor name="sensor_contact" type="contact">
+    <!-- <gazebo reference="${link_name}">
+        <sensor name='sensor_contact' type='contact'>
             <contact>
-                <collision>collision</collision>
+                <collision>wall_collision</collision>
             </contact>
         </sensor>
+    </gazebo> -->
+    <gazebo>
+        <static>true</static>
         <!-- Touch plugin -->
-        <xacro:touch_plugin target="$(arg robot_model_name)" />
-        <!-- <plugin name="gz::sim::systems::TouchPlugin" filename="gz-sim-touchplugin-system">
-                <target>$(arg robot_model_name)</target>
-                <namespace>wall</namespace>
-                <time>0.1</time>
-                <enabled>true</enabled>
-            </plugin> -->
+        <!-- <xacro:touch_plugin target="$(arg robot_model_name)" /> -->
     </gazebo>
 </robot>

Commit message: lidar position fixed

File: gz_models/models/urdf/diff_drive.xacro (robot description, xacro)
@@ -20,5 +20,5 @@
     <xacro:property name="lidar_size" value="0.1" />
     <xacro:property name="lidar_mass" value="0.1" />
-    <xacro:property name="lidar_z_offset" value="0.5" />
+    <xacro:property name="lidar_z_offset" value="0.33" />
     <!-- Wheel Macro -->
     <xacro:macro name="wheel" params="name side">

Commit message: 在小车雷达上方添加了摄像头

File: gz_models/models/urdf/diff_drive.xacro (robot description, xacro)
@@ -144,4 +144,30 @@
         <child link="lidar_link" />
         <origin xyz="0 0 ${lidar_z_offset}" rpy="0 0 0" />
+    </joint>
+    <link name="camera_link">
+        <inertial>
+            <mass value="${lidar_mass}" />
+            <inertia ixx="0.000166667" ixy="0" ixz="0" iyy="0.000166667" iyz="0" izz="0.000166667" />
+        </inertial>
+        <visual>
+            <origin xyz="0 0 0" rpy="0 0 0" />
+            <geometry>
+                <box size="${lidar_size} ${lidar_size} ${lidar_size}" />
+            </geometry>
+            <material name="dark_gray">
+                <color rgba="0.2 0.2 0.2 1" />
+            </material>
+        </visual>
+        <collision>
+            <origin xyz="0 0 0" rpy="0 0 0" />
+            <geometry>
+                <box size="${lidar_size} ${lidar_size} ${lidar_size}" />
+            </geometry>
+        </collision>
+    </link>
+    <joint name="camera_joint" type="fixed">
+        <parent link="lidar_link" />
+        <child link="camera_link" />
+        <origin xyz="0 0 ${lidar_size}" rpy="0 0 0" />
     </joint>
     <!-- Gazebo Plugins -->
@@ -217,3 +243,22 @@
         </sensor>
     </gazebo>
+    <gazebo reference="camera_link">
+        <sensor type="camera" name="top_sensor">
+            <frame_id>$(arg robot_model_name)/camera</frame_id>
+            <camera>
+                <horizontal_fov>1.047</horizontal_fov>
+                <image>
+                    <width>320</width>
+                    <height>240</height>
+                </image>
+                <clip>
+                    <near>0.1</near>
+                    <far>50</far>
+                </clip>
+            </camera>
+            <always_on>1</always_on>
+            <update_rate>30</update_rate>
+            <visualize>true</visualize>
+        </sensor>
+    </gazebo>
 </robot>

Commit message: diff drive robot size modified

File: gz_models/models/urdf/diff_drive.xacro (robot description, xacro)
@@ -6,5 +6,5 @@
     <xacro:property name="chassis_length" value="2.01142" />
     <xacro:property name="chassis_width" value="1" />
-    <xacro:property name="chassis_height" value="0.568726" />
+    <xacro:property name="chassis_height" value="0.268726" />
     <xacro:property name="chassis_mass" value="1.14395" />
     <xacro:property name="wheel_radius" value="0.3" />
@@ -20,5 +20,5 @@
     <xacro:property name="lidar_size" value="0.1" />
     <xacro:property name="lidar_mass" value="0.1" />
-    <xacro:property name="lidar_z_offset" value="0.33" />
+    <xacro:property name="lidar_z_offset" value="0.18" />
     <!-- Wheel Macro -->
     <xacro:macro name="wheel" params="name side">
@@ -143,5 +143,5 @@
         <parent link="chassis" />
         <child link="lidar_link" />
-        <origin xyz="0 0 ${lidar_z_offset}" rpy="0 0 0" />
+        <origin xyz="${chassis_length/2 - lidar_size / 2} 0 ${lidar_z_offset}" rpy="0 0 0" />
     </joint>
     <link name="camera_link">
